File: ece362snakegamepcb/ece362snakegamepcb.kicad_sch (KiCad schematic)
At the start: 50 parts, among them J1 USB_B_Micro, J4 Screw_Terminal_01x02, J5 Conn_ARM_SWD_TagConnect_TC2030, J7 Screw_Terminal_01x02, SW1 SW_Push, SW2 SW_Push, U1 RP2350_80QFN, U2 NCP1117-3.3_SOT223, U3 W25Q128JVS, U4 DNF, U5 24AA025E-SN, Y1 ABM8-272-T3

Commit message: Finished schematic and almost done with PCB layout. Removed autosave file and added several
Parts:
- removed J4: Screw_Terminal_01x02, TerminalBlock_Phoenix:TerminalBlock_Phoenix_MPT-0,5-2-2.54_1x02_P2.54mm_Horizontal, symbol Connector:Screw_Terminal_01x02
- added C23, C27: 100n, Capacitor_SMD:C_0402_1005Metric, symbol Device:C
- added C24, C25, C28: 10u, Capacitor_SMD:C_0805_2012Metric, symbol Device:C
- added C26: 0.1u, Capacitor_SMD:C_0402_1005Metric, symbol Device:C
- added C29: 250u, Capacitor_SMD:C_0402_1005Metric, symbol Device:C
- added C30: 0.05u, Capacitor_SMD:C_0402_1005Metric, symbol Device:C
- added J10, J11, J12: Conn_01x02_Pin, Connector_PinHeader_2.54mm:PinHeader_1x02_P2.54mm_Vertical, symbol Connector:Conn_01x02_Pin
- added J4: Conn_02x08_Counter_Clockwise, Connector_PinHeader_2.54mm:PinHeader_2x08_P2.54mm_Horizontal, symbol Connector_Generic:Conn_02x08_Counter_Clockwise
- added J8: Screw_Terminal_01x02, TerminalBlock_Phoenix:TerminalBlock_Phoenix_MPT-0,5-2-2.54_1x02_P2.54mm_Horizontal, symbol Connector:Screw_Terminal_01x02
- added J9: Conn_01x06_Pin, Connector_PinHeader_2.54mm:PinHeader_1x06_P2.54mm_Horizontal, symbol Connector:Conn_01x06_Pin
- added R12, R14, R15, R16: 4.7k, Resistor_SMD:R_0402_1005Metric, symbol Device:R
- added R17: 1k, Resistor_SMD:R_0402_1005Metric, symbol Device:R
- added R5: 10k, Resistor_SMD:R_0402_1005Metric, symbol Device:R
- added U6: LM1084-5.0, Package_TO_SOT_THT:TO-220-3_Horizontal_TabDown, symbol Regulator_Linear:LM1084-5.0
- added U7: LM324, Package_SO:SSOP-14_5.3x6.2mm_P0.65mm, symbol Amplifier_Operational:LM324
- added U8: LM386, Package_SO:SOIC-8_3.9x4.9mm_P1.27mm, symbol Amplifier_Audio:LM386
Connections:
- net +3.3V: now also C23.1, J10.1 (Pin_1), J10.2 (Pin_2), J9.1 (Pin_1), J9.2 (Pin_2), R15.1, R16.1
- net +3V3: now also R5.1
- net GND: now also U5.1 (A0), U5.2 (A1), U5.3 (A2), U5.7 (WP), C23.2, C24.2, C25.2, C26.2, C27.2, C30.2, J12.2 (Pin_2), J4.13 (Pin_13), J4.15 (Pin_15), J4.9 (Pin_9), J8.1 (Pin_1), J9.5 (Pin_5), J9.6 (Pin_6), R12.2, R14.2, U6.1 (GND), U7.11 (V-), U8.2 (-), U8.4 (GND)
- net GPIO10: now also J4.2 (Pin_2)
- net GPIO11: now also J4.3 (Pin_3)
- net GPIO12: now also J4.14 (Pin_14)
- net GPIO13: now also J4.4 (Pin_4)
- net GPIO14: now also J4.7 (Pin_7)
- net GPIO15: now also J4.10 (Pin_10)
- net GPIO16: now also J4.8 (Pin_8)
- net GPIO17: now also J4.5 (Pin_5)
- net GPIO18: now also J4.12 (Pin_12)
- net GPIO19: now also J4.6 (Pin_6)
- net GPIO20: now also J4.11 (Pin_11)
- net GPIO21: now also J11.1 (Pin_1), R14.1
- net GPIO22: now also J11.2 (Pin_2), R12.1
- net GPIO36: now also R17.2
- net GPIO4: now also U5.5 (SDA), R16.2
- net GPIO40_ADC0: now also J9.3 (Pin_3)
- net GPIO41_ADC1: now also J9.4 (Pin_4)
- net GPIO5: now also U5.6 (SCL), R15.2
- net GPIO8: now also J4.1 (Pin_1)
- net GPIO9: now also J4.16 (Pin_16)
- net VBUS: now also C25.1, C27.1, J8.2 (Pin_2), U6.2 (VO), U7.4 (V+), U8.6 (V+); no longer J7.2 (Pin_2)
- net at J5.3 (~{RESET}): now also R5.2
- new net: C28.1, U8.3 (+)
- new net: C29.2, C30.1, U8.5
- new net: C26.1, R17.1, U7.3 (+)
- new net: C24.1, J7.2 (Pin_2), U6.3 (VI)
- new net: C28.2, U7.1, U7.2 (-)
- new net: C29.1, J12.1 (Pin_1)
Other:
- note added: "Audio"
- note added: "Buttons"
- note added: "Buttons wired off board"
- note added: "Debugger"
- note added: "Joystick (2 axis)"
- note added: "LED Matrix Connections"
- note added: "Main"
- note added: "Screw Terminal VBus (From Battery)"
- note added: "Speaker Pins"
- note added: "To spade connectors (LED Matrix)"
- note removed: "LED Matrix PWR"
- note removed: "Screw Terminal VBus"
- moved on the sheet: C10, C11, C12, C13, C14, C15, C16, C17, C18, C19, C20, C21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

Commit message: Finished pcb layout, but need to fix DRC erros
Parts:
- C29: footprint Capacitor_SMD:C_0402_1005Metric -> Capacitor_THT:C_Radial_D6.3mm_H5.0mm_P2.50mm
- J5: footprint Connector:Tag-Connect_TC2030-IDC-FP_2x03_P1.27mm_Vertical -> Connector:Tag-Connect_TC2030-IDC-NL_2x03_P1.27mm_Vertical
Connections:
- net +3.3V is gone; now on net +3V3: C23.1, J10.1 (Pin_1), J10.2 (Pin_2), J9.1 (Pin_1), J9.2 (Pin_2), R15.1, R16.1, U5.8 (V_{CC})
- net +9V: now reaches C24.1, J7.2 (Pin_2), U6.3 (VI)
Changed lines of the file:
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@@
 	)
 	(junction
+		(at 49.53 358.14)
+		(diameter 0)
+		(color 0 0 0 0)
+	)
+	(junction
 		(at 31.75 336.55)
 		(diameter 0)
@@
 	(wire
 		(pts
-			(xy 41.91 358.14) (xy 50.8 358.14)
+			(xy 41.91 358.14) (xy 49.53 358.14)
 		)
 		(stroke
@@
 	(wire
 		(pts
+			(xy 49.53 358.14) (xy 50.8 358.14)
+		)
+		(stroke
+			(width 0)
+			(type default)
+		)
+	)
+	(wire
+		(pts
 			(xy 256.54 198.12) (xy 271.78 198.12)
 		)
@@
 	)
 	(symbol
+		(lib_id "power:+9V")
+		(at 49.53 358.14 0)
+		(unit 1)
+		(exclude_from_sim no)
+		(in_bom yes)
+		(on_board yes)
+		(dnp no)
+		(fields_autoplaced yes)
+		(property "Reference" "#PWR060"
+			(at 49.53 361.95 0)
+			(effects
+				(font
+					(size 1.27 1.27)
+				)
+				(hide yes)
+			)
+		)
+		(property "Value" "+9V"
+			(at 49.53 353.06 0)
+			(effects
+				(font
+					(size 1.27 1.27)
+				)
+			)
+		)
+		(property "Footprint" ""
+			(at 49.53 358.14 0)
+			(effects
+				(font
+					(size 1.27 1.27)
+				)
+				(hide yes)
+			)
+		)
+		(property "Datasheet" ""
+			(at 49.53 358.14 0)
+			(effects
+				(font
+					(size 1.27 1.27)
+				)
+				(hide yes)
+			)
+		)
+		(property "Description" "Power symbol creates a global label with name \"+9V\""
+			(at 49.53 358.14 0)
+			(effects
+				(font
+					(size 1.27 1.27)
+				)
+				(hide yes)
+			)
+		)
+		(pin "1"
+		)
+		(instances
+			(project ""
+				(path "/94683f5c-9cd9-448e-be96-9792537b5cb8"
+					(reference "#PWR060")
+					(unit 1)
+				)
+			)
+		)
+	)
+	(symbol
 		(lib_id "Amplifier_Audio:LM386")
 		(at 384.81 349.25 0)
@@
 			)
 		)
-		(property "Footprint" "Connector:Tag-Connect_TC2030-IDC-FP_2x03_P1.27mm_Vertical"
+		(property "Footprint" "Connector:Tag-Connect_TC2030-IDC-NL_2x03_P1.27mm_Vertical"
 			(at 60.96 67.31 0)
 			(effects
@@
 			)
 		)
-		(property "Footprint" "Capacitor_SMD:C_0402_1005Metric"
+		(property "Footprint" "Capacitor_THT:C_Radial_D6.3mm_H5.0mm_P2.50mm"
 			(at 398.78 350.2152 0)
 			(effects
@@
 			)
 		)
-		(property "Value" "+3.3V"
+		(property "Value" "+3V3"
 			(at 143.51 308.61 0)
 			(effects
@@
 			)
 		)
-		(property "Value" "+3.3V"
+		(property "Value" "+3V3"
 			(at 219.71 369.57 0)
 			(effects
@@
 			)
 		)
-		(property "Value" "+3.3V"
+		(property "Value" "+3V3"
 			(at 156.21 372.11 0)
 			(effects
@@
 			)
 		)
-		(property "Value" "+3.3V"
+		(property "Value" "+3V3"
 			(at 161.29 308.61 0)
 			(effects

Commit message: Fully completed. added gerbers, bom, placement
Parts:
- removed H1, H2, H3, H4: MountingHole, MountingHole:MountingHole_2.7mm_M2.5, symbol Mechanical:MountingHole
- C22, R11, R13: now not fitted; now left out of the parts list
- U4: footprint Package_SO:SOIC-8_5.23x5.23mm_P1.27mm -> Package_SO:SOIC-8_5.3x5.3mm_P1.27mm; now not fitted; now left out of the parts list
