File: ece362snakegamepcb/ece362snakegamepcb.kicad_pcb (KiCad board)
At the start: 4 copper layers, 53.5 x 54 mm, 69 parts, among them J1 USB_B_Micro, J10 Conn_01x02_Pin, J11 Conn_01x02_Pin, J12 Conn_01x02_Pin, J4 Conn_02x08_Counter_Clockwise, J5 Conn_ARM_SWD_TagConnect_TC2030, J7 Screw_Terminal_01x02, J8 Screw_Terminal_01x02, J9 Conn_01x06_Pin, SW1 SW_Push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

Commit message: Finished PCB for real this time
Parts:
- U6: footprint Package_TO_SOT_THT:TO-220-3_Horizontal_TabDown -> Package_TO_SOT_THT:TO-220-3_Vertical
